File: battery emulator design 0.1/battery emulator design 0.1/battery emulator design 0.1.kicad_pcb (KiCad board)
At the start: 2 copper layers, 205.7 x 66 mm, 88 parts, among them IC1 MAX660CPA, J1 ExtPwrGnd, J10 ExtSetAll, J11 GND_CLIP, J12 V_Out1, J13 ExtPwr, J14 GND, J15 V_Out2, J16 V_Out3, J17 V_Out4, J5 Barrel_Jack, J6 ExtSet1, J7 ExtSet2, J8 ExtSet3, J9 ExtSet4, U1 LM741, U2 LM317_TO-220, U3 LM741, U4 LM317_TO-220, U5 LM741, U6 LM317_TO-220, U7 LM741, U8 LM317_TO-220, U9 L7805

Commit message: added pots to voltage buffers, other minor changes
Parts:
- removed C1, C12, C15, C16, C17, C18, C19, C2, C20, C21, C22, C23, C24, C25, C26, C27, C28, C29, C3, C4: 100nF, Capacitor_THT:C_Disc_D3.4mm_W2.1mm_P2.50mm
- removed C10, C11, C14, C5, C6, C7, C8, C9: 100uF, Capacitor_THT:CP_Radial_D7.5mm_P2.50mm
- removed C13: 220uF, Capacitor_THT:CP_Radial_D10.0mm_P5.00mm
- removed D1: 1N4007, Diode_THT:D_DO-41_SOD81_P10.16mm_Horizontal
- removed F1: 1A, BEL RSTA T1A Fuse:FUSE_RST-1-BULK
- removed H1, H2, H3, H4: MountingHole_Pad, MountingHole:MountingHole_4.3mm_M4_Pad
- removed IC1: MAX660CPA, Package_DIP:DIP-8_W7.62mm_LongPads
- removed J1: ExtPwrGnd, Connector_PinHeader_2.54mm:PinHeader_1x01_P2.54mm_Vertical
- removed J10: ExtSetAll, Connector_PinHeader_2.54mm:PinHeader_1x01_P2.54mm_Vertical
- removed J11: GND_CLIP, Connector_PinHeader_2.54mm:PinHeader_1x04_P2.54mm_Vertical
- removed J12: V_Out1, Connector_PinHeader_2.54mm:PinHeader_1x03_P2.54mm_Vertical
- removed J13: ExtPwr, Connector_PinHeader_2.54mm:PinHeader_1x01_P2.54mm_Vertical
- removed J14: GND, Connector_PinHeader_2.54mm:PinHeader_1x03_P2.54mm_Vertical
- removed J15: V_Out2, Connector_PinHeader_2.54mm:PinHeader_1x03_P2.54mm_Vertical
- removed J16: V_Out3, Connector_PinHeader_2.54mm:PinHeader_1x03_P2.54mm_Vertical
- removed J17: V_Out4, Connector_PinHeader_2.54mm:PinHeader_1x03_P2.54mm_Vertical
- removed J5: Barrel_Jack, Connector_BarrelJack:BarrelJack_Horizontal
- removed J6: ExtSet1, Connector_PinHeader_2.54mm:PinHeader_1x01_P2.54mm_Vertical
- removed J7: ExtSet2, Connector_PinHeader_2.54mm:PinHeader_1x01_P2.54mm_Vertical
- removed J8: ExtSet3, Connector_PinHeader_2.54mm:PinHeader_1x01_P2.54mm_Vertical
- removed J9: ExtSet4, Connector_PinHeader_2.54mm:PinHeader_1x01_P2.54mm_Vertical
- removed JP1, JP2, JP3, JP4, JP5: Jumper_3_Bridged12, Connector_PinHeader_2.54mm:PinHeader_1x03_P2.54mm_Vertical
- removed JP6: SetPot, Connector_PinHeader_2.54mm:PinHeader_1x02_P2.54mm_Vertical
- removed JP7: Preset1, Connector_PinHeader_2.54mm:PinHeader_1x02_P2.54mm_Vertical
- removed JP8: Preset2, Connector_PinHeader_2.54mm:PinHeader_1x02_P2.54mm_Vertical
- removed R10, R15, R20, R5: 120R, Resistor_THT:R_Axial_DIN0207_L6.3mm_D2.5mm_P10.16mm_Horizontal
- removed R11, R12, R13, R14, R16, R17, R18, R19, R6, R7, R8, R9: 100k, Resistor_THT:R_Axial_DIN0207_L6.3mm_D2.5mm_P10.16mm_Horizontal
- removed R21, R22, R23, R24: R_US, Resistor_THT:R_Axial_DIN0207_L6.3mm_D2.5mm_P10.16mm_Horizontal
- removed RV1: 10k, Potentiometer_THT:Potentiometer_Bourns_3386C_Horizontal
- removed U1, U3, U5, U7: LM741, Package_DIP:DIP-8_W7.62mm_LongPads
- removed U2, U4, U6, U8: LM317_TO-220, Package_TO_SOT_THT:TO-220-3_Vertical
- removed U9: L7805, Package_TO_SOT_THT:TO-220-3_Vertical
Routing:
- net VCC: track 265.3 -> 0.00 mm
- net VDC: track 189.7 -> 0.00 mm
- net VEE: track 175.0 -> 0.00 mm
- net +5V: track 95.4 -> 0.00 mm
- net /reg 1/V_out1: track 74.3 -> 0.00 mm, vias 1 -> 0
- net /reg 1/V_Set1: track 54.1 -> 0.00 mm
- net /reg 2/V_out2: track 49.2 -> 0.00 mm
- net /reg 3/V_out3: track 49.2 -> 0.00 mm
- net /reg 4/V_out4: track 42.0 -> 0.00 mm
- net Net-(U3--): track 33.0 -> 0.00 mm
- net Net-(U7--): track 31.3 -> 0.00 mm
- net /reg 2/V_Set2: track 30.9 -> 0.00 mm
- net Net-(U5--): track 29.5 -> 0.00 mm
- net Preset2: track 24.5 -> 0.00 mm
- net Preset1: track 24.4 -> 0.00 mm
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Other:
- board outline removed
- board text removed: "Battery Emulator JMJ '23 MQK '24"
- board text removed: "Cell 1"
- board text removed: "Cell 2"
- board text removed: "Cell 3"
- board text removed: "Cell 4"
- board text removed: "ExtAll"
- board text removed: "ExtSet1 | GlobalSet"
- board text removed: "ExtSet2 | GlobalSet"
- board text removed: "ExtSet3 | GlobalSet"
- board text removed: "ExtSet4 | GlobalSet"
- board text removed: "GND"
- board text removed: "GlobalExtSet | GlobalIntSet"
- board text removed: "SetPot"
- board text removed: "VCC IN"

Commit message: updating with all other boards
Parts:
- added C1: 100nF, Capacitor_THT:C_Disc_D4.3mm_W1.9mm_P5.00mm, F.Cu at (168.9, 76.2)
- added C10: 100uF, Capacitor_THT:CP_Radial_D7.5mm_P2.50mm, F.Cu at (175.3, 118.1)
- added C11: 100uF, Capacitor_THT:CP_Radial_D7.5mm_P2.50mm, F.Cu at (200.7, 118.7)
- added C12: 100nF, Capacitor_THT:C_Disc_D4.3mm_W1.9mm_P5.00mm, F.Cu at (134.0, 76.2)
- added C14: 100uF, Capacitor_THT:CP_Radial_D7.5mm_P2.50mm, F.Cu at (203.8, 79.3)
- added C15: 100nF, Capacitor_THT:C_Disc_D4.3mm_W1.9mm_P5.00mm, F.Cu at (203.8, 64.8)
- added C17: 100nF, Capacitor_THT:C_Disc_D4.3mm_W1.9mm_P5.00mm, F.Cu at (95.9, 76.2)
- added C2: 100nF, Capacitor_THT:C_Disc_D4.3mm_W1.9mm_P5.00mm, F.Cu at (179.7, 95.9)
- added C22: 100nF, Capacitor_THT:C_Disc_D4.3mm_W1.9mm_P5.00mm, F.Cu at (124.4, 125.1)
- added C23: 100nF, Capacitor_THT:C_Disc_D4.3mm_W1.9mm_P5.00mm, F.Cu at (149.8, 125.1)
- added C24: 100nF, Capacitor_THT:C_Disc_D4.3mm_W1.9mm_P5.00mm, F.Cu at (175.2, 125.7)
- added C25: 100nF, Capacitor_THT:C_Disc_D4.3mm_W1.9mm_P5.00mm, F.Cu at (200.6, 125.7)
- added C26: 100nF, Capacitor_THT:C_Disc_D4.3mm_W1.9mm_P5.00mm, F.Cu at (208.9, 109.9)
- added C27: 100nF, Capacitor_THT:C_Disc_D4.3mm_W1.9mm_P5.00mm, F.Cu at (183.5, 109.3)
- added C28: 100nF, Capacitor_THT:C_Disc_D4.3mm_W1.9mm_P5.00mm, F.Cu at (158.1, 109.3)
- added C29: 100nF, Capacitor_THT:C_Disc_D4.3mm_W1.9mm_P5.00mm, F.Cu at (132.7, 109.3)
- added C5: 100uF, Capacitor_THT:CP_Radial_D7.5mm_P2.50mm, F.Cu at (181.6, 67.4)
- added C6: 100uF, Capacitor_THT:CP_Radial_D7.5mm_P2.50mm, F.Cu at (103.5, 76.2)
- added C7: 100uF, Capacitor_THT:CP_Radial_D7.5mm_P2.50mm, F.Cu at (126.4, 76.2)
- added C8: 100uF, Capacitor_THT:CP_Radial_D7.5mm_P2.50mm, F.Cu at (124.5, 117.5)
- added C9: 100uF, Capacitor_THT:CP_Radial_D7.5mm_P2.50mm, F.Cu at (149.9, 118.1)
- added H1: MountingHole_Pad, MountingHole:MountingHole_4.3mm_M4_Pad, F.Cu at (97.3, 67.1)
- added H2: MountingHole_Pad, MountingHole:MountingHole_4.3mm_M4_Pad, F.Cu at (97.3, 132.6)
- added H3: MountingHole_Pad, MountingHole:MountingHole_4.3mm_M4_Pad, F.Cu at (213.6, 67.1)
- added H4: MountingHole_Pad, MountingHole:MountingHole_4.3mm_M4_Pad, F.Cu at (213.6, 132.6)
- added IC1: MAX660CPA, Package_DIP:DIP-8_W7.62mm_LongPads, F.Cu at (190.5, 64.8)
- added J1: Conn_01x08, Connector_PinSocket_2.54mm:PinSocket_1x08_P2.54mm_Vertical, F.Cu at (98.4, 102.9)
- added J12: V_Out1, Connector_PinHeader_2.54mm:PinHeader_1x03_P2.54mm_Vertical, F.Cu at (126.9, 134.0)
- added J15: V_Out2, Connector_PinHeader_2.54mm:PinHeader_1x03_P2.54mm_Vertical, F.Cu at (152.3, 134.0)
- added J16: V_Out3, Connector_PinHeader_2.54mm:PinHeader_1x03_P2.54mm_Vertical, F.Cu at (177.7, 134.0)
- added J17: V_Out4, Connector_PinHeader_2.54mm:PinHeader_1x03_P2.54mm_Vertical, F.Cu at (203.1, 134.0)
- added J2: Conn_01x02_Pin, Connector_PinHeader_2.54mm:PinHeader_1x02_P2.54mm_Vertical, F.Cu at (94.0, 110.5)
- added J3: Conn_01x08, Connector_PinSocket_2.54mm:PinSocket_1x08_P2.54mm_Vertical, F.Cu at (114.3, 102.9)
- added Power_Input1: Conn_01x02_Pin, Connector_PinHeader_2.54mm:PinHeader_1x02_P2.54mm_Vertical, F.Cu at (98.9, 87.0)
- added R1: 10k, Resistor_THT:R_Axial_DIN0207_L6.3mm_D2.5mm_P10.16mm_Horizontal, F.Cu at (116.8, 135.1)
- added R10: 120R, Resistor_THT:R_Axial_DIN0207_L6.3mm_D2.5mm_P10.16mm_Horizontal, F.Cu at (149.9, 99.1)
- added R11: 100k, Resistor_THT:R_Axial_DIN0207_L6.3mm_D2.5mm_P10.16mm_Horizontal, F.Cu at (143.5, 85.1)
- added R12: 100k, Resistor_THT:R_Axial_DIN0207_L6.3mm_D2.5mm_P10.16mm_Horizontal, F.Cu at (127.6, 90.2)
- added R13: 100k, Resistor_THT:R_Axial_DIN0207_L6.3mm_D2.5mm_P10.16mm_Horizontal, F.Cu at (127.6, 95.2)
- added R14: 100k, Resistor_THT:R_Axial_DIN0207_L6.3mm_D2.5mm_P10.16mm_Horizontal, F.Cu at (153.7, 90.2)
- added R15: 120R, Resistor_THT:R_Axial_DIN0207_L6.3mm_D2.5mm_P10.16mm_Horizontal, F.Cu at (175.3, 99.1)
- added R16: 100k, Resistor_THT:R_Axial_DIN0207_L6.3mm_D2.5mm_P10.16mm_Horizontal, F.Cu at (214.0, 99.1)
- added R17: 100k, Resistor_THT:R_Axial_DIN0207_L6.3mm_D2.5mm_P10.16mm_Horizontal, F.Cu at (200.7, 88.9)
- added R18: 100k, Resistor_THT:R_Axial_DIN0207_L6.3mm_D2.5mm_P10.16mm_Horizontal, F.Cu at (200.7, 94.0)
- added R19: 100k, Resistor_THT:R_Axial_DIN0207_L6.3mm_D2.5mm_P10.16mm_Horizontal, F.Cu at (208.3, 88.9)
- added R2: 3.3k, Resistor_THT:R_Axial_DIN0207_L6.3mm_D2.5mm_P10.16mm_Horizontal, F.Cu at (106.7, 124.5)
- added R20: 120R, Resistor_THT:R_Axial_DIN0207_L6.3mm_D2.5mm_P10.16mm_Horizontal, F.Cu at (200.7, 99.1)
- added R21: 3.3k, Resistor_THT:R_Axial_DIN0207_L6.3mm_D2.5mm_P10.16mm_Horizontal, F.Cu at (157.2, 125.0)
- added R22: 10k, Resistor_THT:R_Axial_DIN0207_L6.3mm_D2.5mm_P10.16mm_Horizontal, F.Cu at (167.4, 135.4)
- added R23: 3.3k, Resistor_THT:R_Axial_DIN0207_L6.3mm_D2.5mm_P10.16mm_Horizontal, F.Cu at (182.6, 125.0)
- added R24: 10k, Resistor_THT:R_Axial_DIN0207_L6.3mm_D2.5mm_P10.16mm_Horizontal, F.Cu at (192.8, 135.4)
- added R3: 3.3k, Resistor_THT:R_Axial_DIN0207_L6.3mm_D2.5mm_P10.16mm_Horizontal, F.Cu at (131.9, 125.0)
- added R4: 10k, Resistor_THT:R_Axial_DIN0207_L6.3mm_D2.5mm_P10.16mm_Horizontal, F.Cu at (142.0, 135.4)
- added R5: 820R, Resistor_THT:R_Axial_DIN0207_L6.3mm_D2.5mm_P10.16mm_Horizontal, F.Cu at (124.5, 99.1)
- added R6: 100k, Resistor_THT:R_Axial_DIN0207_L6.3mm_D2.5mm_P10.16mm_Horizontal, F.Cu at (143.5, 80.0)
- added R7: 100k, Resistor_THT:R_Axial_DIN0207_L6.3mm_D2.5mm_P10.16mm_Horizontal, F.Cu at (143.5, 64.8)
- added R8: 100k, Resistor_THT:R_Axial_DIN0207_L6.3mm_D2.5mm_P10.16mm_Horizontal, F.Cu at (143.5, 69.8)
- added R9: 100k, Resistor_THT:R_Axial_DIN0207_L6.3mm_D2.5mm_P10.16mm_Horizontal, F.Cu at (153.7, 74.9)
- added RV2: 10k, battery_emulator:PDB181, F.Cu at (111.7, 130.2)
- added RV3: 10k, battery_emulator:PDB181, F.Cu at (137.0, 130.2)
- added RV4: 10k, battery_emulator:PDB181, F.Cu at (162.4, 130.2)
- added RV5: 10k, battery_emulator:PDB181, F.Cu at (187.8, 130.2)
- added U1: LM324, Package_DIP:DIP-14_W7.62mm_LongPads, F.Cu at (176.5, 81.3)
- added U2: LM317_TO-220, Package_TO_SOT_THT:TO-220-3_Vertical, F.Cu at (121.9, 109.2)
- added U4: LM317_TO-220, Package_TO_SOT_THT:TO-220-3_Vertical, F.Cu at (147.3, 109.2)
- added U6: LM317_TO-220, Package_TO_SOT_THT:TO-220-3_Vertical, F.Cu at (172.7, 109.2)
- added U8: LM317_TO-220, Package_TO_SOT_THT:TO-220-3_Vertical, F.Cu at (198.1, 109.5)
- added U9: L7805, Package_TO_SOT_THT:TO-220-3_Vertical, F.Cu at (112.4, 78.4)
Routing:
- net +5V: track 0.00 -> 152.3 mm, vias 0 -> 3
- net /reg 1/V_out1: track 0.00 -> 137.1 mm
- net V_Set_4: track 0.00 -> 126.9 mm, vias 0 -> 2
- net V_Set_1: track 0.00 -> 126.4 mm
- net /reg 3/V_out3: track 0.00 -> 120.6 mm
- net VCC: track 0.00 -> 115.1 mm, vias 0 -> 2
- net /reg 2/V_out2: track 0.00 -> 102.5 mm
- net Net-(U2-ADJ): track 0.00 -> 100.3 mm, vias 0 -> 3
- net /SurfBoard/S4A: track 0.00 -> 90.0 mm, vias 0 -> 2
- net V_Set_2: track 0.00 -> 83.0 mm
- net Net-(U8-ADJ): track 0.00 -> 61.0 mm
- net /SurfBoard/S3A: track 0.00 -> 58.8 mm
- net Net-(U4-ADJ): track 0.00 -> 57.9 mm
- net Net-(U1D--): track 0.00 -> 51.6 mm
- net /SurfBoard/S2A: track 0.00 -> 49.3 mm
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- added copper zone on F.Cu, net +5V
- added copper zone on B.Cu, net GND
- added copper zone on F.Cu, net VCC
- added copper zone on F.Cu, net VEE
Other:
- board outline added: 127 x 76.2 mm
- board text added: "GND"
- board text added: "SW"
- board text added: "TRCK"
- board text added: "VCC"
