File: battery emulator design 0.1/battery emulator design 0.1/power.kicad_sch (KiCad schematic)
At the start: 14 parts, among them IC1 MAX660CPA, J13 ExtPwr, J5 Barrel_Jack, U9 L7805

Commit message: updating with all other boards
Parts:
- removed C13: 220uF, Capacitor_THT:CP_Radial_D10.0mm_P5.00mm, symbol Device:C_Polarized
- removed D1: 1N4007, Diode_THT:D_DO-41_SOD81_P10.16mm_Horizontal, symbol Diode:1N4007
- removed F1: 1A, BEL RSTA T1A Fuse:FUSE_RST-1-BULK, symbol Device:Fuse
- removed J13: ExtPwr, Connector_PinHeader_2.54mm:PinHeader_1x01_P2.54mm_Vertical, symbol Connector:Conn_01x01_Pin
- removed J5: Barrel_Jack, Connector_BarrelJack:BarrelJack_Horizontal, symbol Connector:Barrel_Jack
- added Power_Input1: Conn_01x02_Pin, Connector_PinHeader_2.54mm:PinHeader_1x02_P2.54mm_Vertical, symbol Connector:Conn_01x02_Pin
- C12, C15, C17: footprint Capacitor_THT:C_Disc_D3.4mm_W2.1mm_P2.50mm -> Capacitor_THT:C_Disc_D4.3mm_W1.9mm_P5.00mm
Connections:
- net GND: now also Power_Input1.2 (Pin_2)
- net VCC: now also Power_Input1.1 (Pin_1)
Other:
- note removed: "24 V - 30 V DC"
